Commit message: visualise

File: urdf/robot.urdf (robot description, URDF)
Before this commit: robot Bot1, 13 links, 12 joints
Links:
- added link floor; collision box size=10 10 0.1; visual box size=10 10 0.1
- added link world
- link part_1: geometry collision mesh filename=part_1.stl; visual mesh filename=part_1.stl
- link part_1_10: geometry collision mesh filename=part_1__4.stl; visual mesh filename=part_1__4.stl
- link part_1_11: geometry collision mesh filename=part_1__2.stl; visual mesh filename=part_1__2.stl
- link part_1_12: geometry collision mesh filename=part_1__3.stl; visual mesh filename=part_1__3.stl
- link part_1_13: geometry collision mesh filename=part_1__4.stl; visual mesh filename=part_1__4.stl
- link part_1_2: geometry collision mesh filename=part_1__2.stl; visual mesh filename=part_1__2.stl
- link part_1_3: geometry collision mesh filename=part_1__3.stl; visual mesh filename=part_1__3.stl
- link part_1_4: geometry collision mesh filename=part_1__4.stl; visual mesh filename=part_1__4.stl
- link part_1_5: geometry collision mesh filename=part_1__2.stl; visual mesh filename=part_1__2.stl
- link part_1_6: geometry collision mesh filename=part_1__3.stl; visual mesh filename=part_1__3.stl
- link part_1_7: geometry collision mesh filename=part_1__4.stl; visual mesh filename=part_1__4.stl
- link part_1_8: geometry collision mesh filename=part_1__2.stl; visual mesh filename=part_1__2.stl
- link part_1_9: geometry collision mesh filename=part_1__3.stl; visual mesh filename=part_1__3.stl
Joints:
- added joint floor_to_base: type floating, parent floor, child part_1, origin xyz=0 0 0.5 rpy=0 0 0
- added joint world_to_floor: type fixed, parent world, child floor, origin xyz=0 0 0 rpy=0 0 0

Commit message: improved reward functions

File: urdf/robot.urdf (robot description, URDF)
Before this commit: robot Bot1, 15 links, 14 joints
Joints:
- joint floor_to_base: origin xyz=0 0 0.5 rpy=0 0 0 -> xyz=0 0 0.2 rpy=0 0 0
